Commit message: 完成惯性和质量的添加

File: chapt6/chapt6_ws/install/fishbot_description/share/fishbot_description/urdf/fishbot/actuator/caster.urdf.xacro (robot description, xacro)
@@ -1,29 +1,31 @@
 <?xml version="1.0"?>
 <robot xmlns:xacro="http://www.ros.org/wiki/xacro">
+    <xacro:include filename="$(find fishbot_description)/urdf/fishbot/common_inertia.urdf.xacro" />
     <xacro:macro name="caster_xacro" params="caster_name xyz">
         <link name="${caster_name}_link">
             <visual>
-                <origin xyz="0.0 0.0 0.0" rpy="1.57079 0.0 0.0"/>
+                <origin xyz="0.0 0.0 0.0" rpy="1.57079 0.0 0.0" />
                 <geometry>
-                    <sphere radius="0.016"/>
+                    <sphere radius="0.016" />
                 </geometry>
                 <material name="yellow">
-                    <color rgba="1.0 1.0 0 0.8"/>
+                    <color rgba="1.0 1.0 0 0.8" />
                 </material>
             </visual>
             <collision>
-                <origin xyz="0.0 0.0 0.0" rpy="1.57079 0.0 0.0"/>
+                <origin xyz="0.0 0.0 0.0" rpy="1.57079 0.0 0.0" />
                 <geometry>
-                    <sphere radius="0.016"/>
+                    <sphere radius="0.016" />
                 </geometry>
                 <material name="yellow">
-                    <color rgba="1.0 1.0 0 0.8"/>
+                    <color rgba="1.0 1.0 0 0.8" />
                 </material>
             </collision>
+            <xacro:sphere_inertia m="0.05" r="0.016" />
         </link>
         <joint name="${caster_name}_base_link_joint" type="fixed">
-            <parent link="base_link"/>
-            <child link="${caster_name}_link"/>
-            <origin xyz="${xyz}" rpy="0.0 0.0 0.0"/>
+            <parent link="base_link" />
+            <child link="${caster_name}_link" />
+            <origin xyz="${xyz}" rpy="0.0 0.0 0.0" />
         </joint>
     </xacro:macro>

File: chapt6/chapt6_ws/install/fishbot_description/share/fishbot_description/urdf/fishbot/actuator/wheel.urdf.xacro (robot description, xacro)
@@ -1,30 +1,32 @@
 <?xml version="1.0"?>
 <robot xmlns:xacro="http://www.ros.org/wiki/xacro">
+    <xacro:include filename="$(find fishbot_description)/urdf/fishbot/common_inertia.urdf.xacro" />
     <xacro:macro name="wheel_xacro" params="wheel_name xyz">
         <link name="${wheel_name}_link">
             <visual>
-                <origin xyz="0.0 0.0 0.0" rpy="1.57079 0.0 0.0"/>
+                <origin xyz="0.0 0.0 0.0" rpy="1.57079 0.0 0.0" />
                 <geometry>
-                    <cylinder radius="0.032" length="0.04"/>
+                    <cylinder radius="0.032" length="0.04" />
                 </geometry>
                 <material name="yellow">
-                    <color rgba="1.0 1.0 0 0.8"/>
+                    <color rgba="1.0 1.0 0 0.8" />
                 </material>
             </visual>
             <collision>
-                <origin xyz="0.0 0.0 0.0" rpy="1.57079 0.0 0.0"/>
+                <origin xyz="0.0 0.0 0.0" rpy="1.57079 0.0 0.0" />
                 <geometry>
-                    <cylinder radius="0.032" length="0.04"/>
+                    <cylinder radius="0.032" length="0.04" />
                 </geometry>
                 <material name="yellow">
-                    <color rgba="1.0 1.0 0 0.8"/>
+                    <color rgba="1.0 1.0 0 0.8" />
                 </material>
             </collision>
+            <xacro:cylinder_inertia m="0.05" r="0.032" h="0.04" />
         </link>
         <joint name="${wheel_name}_base_link_joint" type="continuous">
-            <parent link="base_link"/>
-            <child link="${wheel_name}_link"/>
-            <origin xyz="${xyz}" rpy="0.0 0.0 0.0"/>
-            <axis xyz="0 1 0"/>
+            <parent link="base_link" />
+            <child link="${wheel_name}_link" />
+            <origin xyz="${xyz}" rpy="0.0 0.0 0.0" />
+            <axis xyz="0 1 0" />
         </joint>
     </xacro:macro>

File: chapt6/chapt6_ws/install/fishbot_description/share/fishbot_description/urdf/fishbot/base.urdf.xacro (robot description, xacro)
@@ -1,32 +1,32 @@
 <?xml version="1.0"?>
 <robot xmlns:xacro="http://www.ros.org/wiki/xacro">
-    <xacro:include filename="$(find fishbot_description)/urdf/fishbot/common_inertia.urdf.xacro"/>
+    <xacro:include filename="$(find fishbot_description)/urdf/fishbot/common_inertia.urdf.xacro" />
     <xacro:macro name="base_xacro" params="length radius">
-        <link name="base_foot_print"/>
+        <link name="base_foot_print" />
         <link name="base_link">
             <visual>
-                <origin xyz="0.0 0.0 0.0" rpy="0.0 0.0 0.0"/>
+                <origin xyz="0.0 0.0 0.0" rpy="0.0 0.0 0.0" />
                 <geometry>
-                    <cylinder radius="${radius}" length="${length}"/>
+                    <cylinder radius="${radius}" length="${length}" />
                 </geometry>
                 <material name="white">
-                    <color rgba="1.0 1.0 1.0 0.5"/>
+                    <color rgba="1.0 1.0 1.0 0.5" />
                 </material>
             </visual>
             <collision>
-                <origin xyz="0.0 0.0 0.0" rpy="0.0 0.0 0.0"/>
+                <origin xyz="0.0 0.0 0.0" rpy="0.0 0.0 0.0" />
                 <geometry>
-                    <cylinder radius="${radius}" length="${length}"/>
+                    <cylinder radius="${radius}" length="${length}" />
                 </geometry>
                 <material name="white">
-                    <color rgba="1.0 1.0 1.0 0.5"/>
+                    <color rgba="1.0 1.0 1.0 0.5" />
                 </material>
             </collision>
-            <xacro:cylinder_inertia m="1.0" r="${radius}" h="${length}"/>
+            <xacro:cylinder_inertia m="1.0" r="${radius}" h="${length}" />
         </link>
         <joint name="base_to_footprint_joint" type="fixed">
-            <origin xyz="0.0 0.0 ${length/2+0.032-0.001}" rpy="0.0 0.0 0.0"/>
-            <parent link="base_foot_print"/>
-            <child link="base_link"/>
+            <origin xyz="0.0 0.0 ${length/2+0.032-0.001}" rpy="0.0 0.0 0.0" />
+            <parent link="base_foot_print" />
+            <child link="base_link" />
         </joint>
     </xacro:macro>

File: chapt6/chapt6_ws/install/fishbot_description/share/fishbot_description/urdf/fishbot/fishbot.urdf.xacro (robot description, xacro)
@@ -1,17 +1,17 @@
 <?xml version="1.0"?>
 <robot xmlns:xacro="http://www.ros.org/wiki/xacro" name="fishbot">
-    <xacro:include filename="$(find fishbot_description)/urdf/fishbot/base.urdf.xacro"/>
-    <xacro:include filename="$(find fishbot_description)/urdf/fishbot/sensor/camera.urdf.xacro"/>
-    <xacro:include filename="$(find fishbot_description)/urdf/fishbot/sensor/laser.urdf.xacro"/>
-    <xacro:include filename="$(find fishbot_description)/urdf/fishbot/sensor/imu.urdf.xacro"/>
-    <xacro:include filename="$(find fishbot_description)/urdf/fishbot/actuator/wheel.urdf.xacro"/>
-    <xacro:include filename="$(find fishbot_description)/urdf/fishbot/actuator/caster.urdf.xacro"/>
-    <xacro:base_xacro length="0.12" radius="0.1"/>
-    <xacro:imu_xacro xyz="0 0 0.02"/>
-    <xacro:camera_xacro xyz="0.10 0.0 0.075"/>
-    <xacro:laser_xacro xyz="0 0 0.10"/>
-    <xacro:wheel_xacro wheel_name="left" xyz="0 0.10 -0.06"/>
-    <xacro:wheel_xacro wheel_name="right" xyz="0 -0.10 -0.06"/>
-    <xacro:caster_xacro caster_name="front_caster" xyz="0.08 0 -0.076"/>
-    <xacro:caster_xacro caster_name="back_caster" xyz="-0.08 0 -0.076"/>
+    <xacro:include filename="$(find fishbot_description)/urdf/fishbot/base.urdf.xacro" />
+    <xacro:include filename="$(find fishbot_description)/urdf/fishbot/sensor/camera.urdf.xacro" />
+    <xacro:include filename="$(find fishbot_description)/urdf/fishbot/sensor/laser.urdf.xacro" />
+    <xacro:include filename="$(find fishbot_description)/urdf/fishbot/sensor/imu.urdf.xacro" />
+    <xacro:include filename="$(find fishbot_description)/urdf/fishbot/actuator/wheel.urdf.xacro" />
+    <xacro:include filename="$(find fishbot_description)/urdf/fishbot/actuator/caster.urdf.xacro" />
+    <xacro:base_xacro length="0.12" radius="0.1" />
+    <xacro:imu_xacro xyz="0 0 0.02" />
+    <xacro:camera_xacro xyz="0.10 0.0 0.075" />
+    <xacro:laser_xacro xyz="0 0 0.10" />
+    <xacro:wheel_xacro wheel_name="left" xyz="0 0.10 -0.06" />
+    <xacro:wheel_xacro wheel_name="right" xyz="0 -0.10 -0.06" />
+    <xacro:caster_xacro caster_name="front_caster" xyz="0.08 0 -0.076" />
+    <xacro:caster_xacro caster_name="back_caster" xyz="-0.08 0 -0.076" />
 </robot>

File: chapt6/chapt6_ws/install/fishbot_description/share/fishbot_description/urdf/fishbot/sensor/camera.urdf.xacro (robot description, xacro)
@@ -1,4 +1,5 @@
 <?xml version="1.0"?>
 <robot xmlns:xacro="http://www.ros.org/wiki/xacro">
+    <xacro:include filename="$(find fishbot_description)/urdf/fishbot/common_inertia.urdf.xacro" />
     <xacro:macro name="camera_xacro" params="xyz">
         <link name="camera_link">
@@ -21,4 +22,5 @@
                 </material>
             </collision>
+            <xacro:box_inertia m="0.1" w="0.02" h="0.10" d="0.02" />
         </link>
         <!-- 关节用于组合部件 -->

File: chapt6/chapt6_ws/install/fishbot_description/share/fishbot_description/urdf/fishbot/sensor/imu.urdf.xacro (robot description, xacro)
@@ -1,4 +1,5 @@
 <?xml version="1.0"?>
 <robot xmlns:xacro="http://www.ros.org/wiki/xacro">
+    <xacro:include filename="$(find fishbot_description)/urdf/fishbot/common_inertia.urdf.xacro" />
     <xacro:macro name="imu_xacro" params="xyz">
         <link name="imu_link">
@@ -12,4 +13,11 @@
                 </material>
             </visual>
+            <collision>
+                <origin xyz="0.0 0.0 0.0" rpy="0.0 0.0 0.0" />
+                <geometry>
+                    <box size="0.02 0.02 0.02" />
+                </geometry>
+            </collision>
+            <xacro:box_inertia m="0.05" w="0.02" h="0.02" d="0.02" />
         </link>
         <!-- 关节用于组合部件 -->

File: chapt6/chapt6_ws/install/fishbot_description/share/fishbot_description/urdf/fishbot/sensor/laser.urdf.xacro (robot description, xacro)
@@ -1,25 +1,27 @@
 <?xml version="1.0"?>
 <robot xmlns:xacro="http://www.ros.org/wiki/xacro">
+    <xacro:include filename="$(find fishbot_description)/urdf/fishbot/common_inertia.urdf.xacro" />
     <xacro:macro name="laser_xacro" params="xyz">
         <!-- 雷达支撑杆 -->
         <link name="laser_cylinder_link">
             <visual>
-                <origin xyz="0 0 0" rpy="0 0 0"/>
+                <origin xyz="0 0 0" rpy="0 0 0" />
                 <geometry>
-                    <cylinder radius="0.01" length="0.10"/>
+                    <cylinder radius="0.01" length="0.10" />
                 </geometry>
                 <material name="black">
-                    <color rgba="0 0 0 1"/>
+                    <color rgba="0 0 0 1" />
                 </material>
             </visual>
             <collision>
-                <origin xyz="0 0 0" rpy="0 0 0"/>
+                <origin xyz="0 0 0" rpy="0 0 0" />
                 <geometry>
-                    <cylinder radius="0.01" length="0.10"/>
+                    <cylinder radius="0.01" length="0.10" />
                 </geometry>
                 <material name="black">
-                    <color rgba="0 0 0 1"/>
+                    <color rgba="0 0 0 1" />
                 </material>
             </collision>
+            <xacro:cylinder_inertia m="0.05" r="0.01" h="0.10" />
         </link>
         <link name="laser_link">
@@ -27,5 +29,5 @@
                 <origin xyz="0.0 0.0 0.0" rpy="0.0 0.0 0.0" />
                 <geometry>
-                    <cylinder radius="0.02" length="0.02"/>
+                    <cylinder radius="0.02" length="0.02" />
                 </geometry>
                 <material name="black">
@@ -36,5 +38,5 @@
                 <origin xyz="0.0 0.0 0.0" rpy="0.0 0.0 0.0" />
                 <geometry>
-                    <cylinder radius="0.02" length="0.02"/>
+                    <cylinder radius="0.02" length="0.02" />
                 </geometry>
                 <material name="black">
@@ -42,10 +44,11 @@
                 </material>
             </collision>
+            <xacro:cylinder_inertia m="0.10" r="0.02" h="0.02" />
         </link>
         <!-- 关节用于组合部件 -->
         <joint name="laser_cylinder_joint" type="fixed">
-            <parent link="laser_cylinder_link"/>
-            <child link="laser_link"/>
-            <origin xyz="0.0 0.0 0.05" rpy="0.0 0.0 0.0"/>
+            <parent link="laser_cylinder_link" />
+            <child link="laser_link" />
+            <origin xyz="0.0 0.0 0.05" rpy="0.0 0.0 0.0" />
         </joint>
         <joint name="laser_cylinder_base_link_joint" type="fixed">

File: chapt6/chapt6_ws/src/fishbot_description/urdf/fishbot/actuator/caster.urdf.xacro (robot description, xacro)
@@ -1,31 +1,31 @@
 <?xml version="1.0"?>
 <robot xmlns:xacro="http://www.ros.org/wiki/xacro">
-    <xacro:include filename="$(find fishbot_description)/urdf/fishbot/common_inertia.urdf.xacro"/>
+    <xacro:include filename="$(find fishbot_description)/urdf/fishbot/common_inertia.urdf.xacro" />
     <xacro:macro name="caster_xacro" params="caster_name xyz">
         <link name="${caster_name}_link">
             <visual>
-                <origin xyz="0.0 0.0 0.0" rpy="1.57079 0.0 0.0"/>
+                <origin xyz="0.0 0.0 0.0" rpy="1.57079 0.0 0.0" />
                 <geometry>
-                    <sphere radius="0.016"/>
+                    <sphere radius="0.016" />
                 </geometry>
                 <material name="yellow">
-                    <color rgba="1.0 1.0 0 0.8"/>
+                    <color rgba="1.0 1.0 0 0.8" />
                 </material>
             </visual>
             <collision>
-                <origin xyz="0.0 0.0 0.0" rpy="1.57079 0.0 0.0"/>
+                <origin xyz="0.0 0.0 0.0" rpy="1.57079 0.0 0.0" />
                 <geometry>
-                    <sphere radius="0.016"/>
+                    <sphere radius="0.016" />
                 </geometry>
                 <material name="yellow">
-                    <color rgba="1.0 1.0 0 0.8"/>
+                    <color rgba="1.0 1.0 0 0.8" />
                 </material>
             </collision>
-            <xacro:shpere_inertia m="0.05" r="0.016"/>
+            <xacro:sphere_inertia m="0.05" r="0.016" />
         </link>
         <joint name="${caster_name}_base_link_joint" type="fixed">
-            <parent link="base_link"/>
-            <child link="${caster_name}_link"/>
-            <origin xyz="${xyz}" rpy="0.0 0.0 0.0"/>
+            <parent link="base_link" />
+            <child link="${caster_name}_link" />
+            <origin xyz="${xyz}" rpy="0.0 0.0 0.0" />
         </joint>
     </xacro:macro>

File: chapt6/chapt6_ws/src/fishbot_description/urdf/fishbot/actuator/wheel.urdf.xacro (robot description, xacro)
@@ -1,32 +1,32 @@
 <?xml version="1.0"?>
 <robot xmlns:xacro="http://www.ros.org/wiki/xacro">
-    <xacro:include filename="$(find fishbot_description)/urdf/fishbot/common_inertia.urdf.xacro"/>
+    <xacro:include filename="$(find fishbot_description)/urdf/fishbot/common_inertia.urdf.xacro" />
     <xacro:macro name="wheel_xacro" params="wheel_name xyz">
         <link name="${wheel_name}_link">
             <visual>
-                <origin xyz="0.0 0.0 0.0" rpy="1.57079 0.0 0.0"/>
+                <origin xyz="0.0 0.0 0.0" rpy="1.57079 0.0 0.0" />
                 <geometry>
-                    <cylinder radius="0.032" length="0.04"/>
+                    <cylinder radius="0.032" length="0.04" />
                 </geometry>
                 <material name="yellow">
-                    <color rgba="1.0 1.0 0 0.8"/>
+                    <color rgba="1.0 1.0 0 0.8" />
                 </material>
             </visual>
             <collision>
-                <origin xyz="0.0 0.0 0.0" rpy="1.57079 0.0 0.0"/>
+                <origin xyz="0.0 0.0 0.0" rpy="1.57079 0.0 0.0" />
                 <geometry>
-                    <cylinder radius="0.032" length="0.04"/>
+                    <cylinder radius="0.032" length="0.04" />
                 </geometry>
                 <material name="yellow">
-                    <color rgba="1.0 1.0 0 0.8"/>
+                    <color rgba="1.0 1.0 0 0.8" />
                 </material>
             </collision>
-            <xacro:cylinder_inertia m="0.05" r="0.032" h="0.04"/>
+            <xacro:cylinder_inertia m="0.05" r="0.032" h="0.04" />
         </link>
         <joint name="${wheel_name}_base_link_joint" type="continuous">
-            <parent link="base_link"/>
-            <child link="${wheel_name}_link"/>
-            <origin xyz="${xyz}" rpy="0.0 0.0 0.0"/>
-            <axis xyz="0 1 0"/>
+            <parent link="base_link" />
+            <child link="${wheel_name}_link" />
+            <origin xyz="${xyz}" rpy="0.0 0.0 0.0" />
+            <axis xyz="0 1 0" />
         </joint>
     </xacro:macro>

File: chapt6/chapt6_ws/src/fishbot_description/urdf/fishbot/sensor/camera.urdf.xacro (robot description, xacro)
@@ -1,5 +1,5 @@
 <?xml version="1.0"?>
 <robot xmlns:xacro="http://www.ros.org/wiki/xacro">
-    <xacro:include filename="$(find fishbot_description)/urdf/fishbot/common_inertia.urdf.xacro"/>
+    <xacro:include filename="$(find fishbot_description)/urdf/fishbot/common_inertia.urdf.xacro" />
     <xacro:macro name="camera_xacro" params="xyz">
         <link name="camera_link">
@@ -22,5 +22,5 @@
                 </material>
             </collision>
-            <xacro:box_inertia m="0.1" w="0.02" h="0.10" d="0.02"/>
+            <xacro:box_inertia m="0.1" w="0.02" h="0.10" d="0.02" />
         </link>
         <!-- 关节用于组合部件 -->

File: chapt6/chapt6_ws/src/fishbot_description/urdf/fishbot/sensor/imu.urdf.xacro (robot description, xacro)
@@ -1,5 +1,5 @@
 <?xml version="1.0"?>
 <robot xmlns:xacro="http://www.ros.org/wiki/xacro">
-    <xacro:include filename="$(find fishbot_description)/urdf/fishbot/common_inertia.urdf.xacro"/>
+    <xacro:include filename="$(find fishbot_description)/urdf/fishbot/common_inertia.urdf.xacro" />
     <xacro:macro name="imu_xacro" params="xyz">
         <link name="imu_link">
@@ -13,16 +13,11 @@
                 </material>
             </visual>
-        <collision>
-            <visual>
+            <collision>
                 <origin xyz="0.0 0.0 0.0" rpy="0.0 0.0 0.0" />
                 <geometry>
                     <box size="0.02 0.02 0.02" />
                 </geometry>
-                <material name="black">
-                    <color rgba="0.0 0.0 0.0 1.0" />
-                </material>
-            </visual>
-        </collision>
-        <xacro:box_inertia m="0.05" w="0.02" h="0.02" d="0.02"/>
+            </collision>
+            <xacro:box_inertia m="0.05" w="0.02" h="0.02" d="0.02" />
         </link>
         <!-- 关节用于组合部件 -->

File: chapt6/chapt6_ws/src/fishbot_description/urdf/fishbot/sensor/laser.urdf.xacro (robot description, xacro)
@@ -1,26 +1,27 @@
 <?xml version="1.0"?>
 <robot xmlns:xacro="http://www.ros.org/wiki/xacro">
-    <xacro:include filename="$(find fishbot_description)/urdf/fishbot/common_inertia.urdf.xacro"/>
+    <xacro:include filename="$(find fishbot_description)/urdf/fishbot/common_inertia.urdf.xacro" />
     <xacro:macro name="laser_xacro" params="xyz">
         <!-- 雷达支撑杆 -->
         <link name="laser_cylinder_link">
             <visual>
-                <origin xyz="0 0 0" rpy="0 0 0"/>
+                <origin xyz="0 0 0" rpy="0 0 0" />
                 <geometry>
-                    <cylinder radius="0.01" length="0.10"/>
+                    <cylinder radius="0.01" length="0.10" />
                 </geometry>
                 <material name="black">
-                    <color rgba="0 0 0 1"/>
+                    <color rgba="0 0 0 1" />
                 </material>
             </visual>
             <collision>
-                <origin xyz="0 0 0" rpy="0 0 0"/>
+                <origin xyz="0 0 0" rpy="0 0 0" />
                 <geometry>
-                    <cylinder radius="0.01" length="0.10"/>
+                    <cylinder radius="0.01" length="0.10" />
                 </geometry>
                 <material name="black">
-                    <color rgba="0 0 0 1"/>
+                    <color rgba="0 0 0 1" />
                 </material>
             </collision>
+            <xacro:cylinder_inertia m="0.05" r="0.01" h="0.10" />
         </link>
         <link name="laser_link">
@@ -28,5 +29,5 @@
                 <origin xyz="0.0 0.0 0.0" rpy="0.0 0.0 0.0" />
                 <geometry>
-                    <cylinder radius="0.02" length="0.02"/>
+                    <cylinder radius="0.02" length="0.02" />
                 </geometry>
                 <material name="black">
@@ -37,5 +38,5 @@
                 <origin xyz="0.0 0.0 0.0" rpy="0.0 0.0 0.0" />
                 <geometry>
-                    <cylinder radius="0.02" length="0.02"/>
+                    <cylinder radius="0.02" length="0.02" />
                 </geometry>
                 <material name="black">
@@ -43,10 +44,11 @@
                 </material>
             </collision>
+            <xacro:cylinder_inertia m="0.10" r="0.02" h="0.02" />
         </link>
         <!-- 关节用于组合部件 -->
         <joint name="laser_cylinder_joint" type="fixed">
-            <parent link="laser_cylinder_link"/>
-            <child link="laser_link"/>
-            <origin xyz="0.0 0.0 0.05" rpy="0.0 0.0 0.0"/>
+            <parent link="laser_cylinder_link" />
+            <child link="laser_link" />
+            <origin xyz="0.0 0.0 0.05" rpy="0.0 0.0 0.0" />
         </joint>
         <joint name="laser_cylinder_base_link_joint" type="fixed">
