Commit message: 学习gazebo中urdf扩展添加

File: chapt6/chapt6_ws/install/fishbot_description/share/fishbot_description/urdf/fishbot/actuator/caster.urdf.xacro (robot description, xacro)
@@ -29,4 +29,11 @@
             <origin xyz="${xyz}" rpy="0.0 0.0 0.0" />
         </joint>
+        <gazebo reference="${caster_name}_link">
+            <mu1 value="0.0"/>
+            <mu2 value="0.0"/>
+            <kp value="1000000000.0"/>
+            <kd value="1.0"/>
+            <material>Gazebo/Yellow</material>
+        </gazebo>
     </xacro:macro>
 </robot>

File: chapt6/chapt6_ws/install/fishbot_description/share/fishbot_description/urdf/fishbot/actuator/wheel.urdf.xacro (robot description, xacro)
@@ -30,4 +30,13 @@
             <axis xyz="0 1 0" />
         </joint>
+        <gazebo reference="${wheel_name}_link">
+            <mu1 value="20.0"/>
+            <mu2 value="20.0"/>
+            <kp value="1000000000.0"/>
+            <kd value="1.0"/>
+            <material>
+                Gazebo/Yellow
+            </material>
+        </gazebo>
     </xacro:macro>
 </robot>

File: chapt6/chapt6_ws/install/fishbot_description/share/fishbot_description/urdf/fishbot/sensor/camera.urdf.xacro (robot description, xacro)
@@ -30,4 +30,7 @@
             <origin xyz="${xyz}" rpy="0.0 0.0 0.0" />
         </joint>
+        <gazebo reference="camera_link">
+            <material>Gazebo/Black</material>
+        </gazebo>
     </xacro:macro>
 </robot>

File: chapt6/chapt6_ws/install/fishbot_description/share/fishbot_description/urdf/fishbot/sensor/laser.urdf.xacro (robot description, xacro)
@@ -57,4 +57,10 @@
             <origin xyz="${xyz}" rpy="0.0 0.0 0.0" />
         </joint>
+        <gazebo reference="laser_cylinder_link">
+            <material>Gazebo/Black</material>
+        </gazebo>
+        <gazebo reference="laser_link">
+            <material>Gazebo/Black</material>
+        </gazebo>
     </xacro:macro>
 </robot>
