Commit message: 添加地面坐标系

File: chapt6/chapt6_ws/install/fishbot_description/share/fishbot_description/urdf/fishbot/base.urdf.xacro (robot description, xacro)
@@ -2,4 +2,5 @@
 <robot xmlns:xacro="http://www.ros.org/wiki/xacro">
     <xacro:macro name="base_xacro" params="length radius">
+        <link name="base_foot_print"/>
         <link name="base_link">
             <visual>
@@ -13,4 +14,9 @@
             </visual>
         </link>
+        <joint name="base_to_footprint_joint" type="fixed">
+            <origin xyz="0.0 0.0 ${length/2+0.032-0.001}" rpy="0.0 0.0 0.0"/>
+            <parent link="base_foot_print"/>
+            <child link="base_link"/>
+        </joint>
     </xacro:macro>
 </robot>

Commit message: claude修改之前的副本

File: chapt6/chapt6_ws/install/fishbot_description/share/fishbot_description/urdf/fishbot/base.urdf.xacro (robot description, xacro)
@@ -1,4 +1,5 @@
 <?xml version="1.0"?>
 <robot xmlns:xacro="http://www.ros.org/wiki/xacro">
+    <xacro:include filename="$(find fishbot_description)/urdf/fishbot/common_inertia.urdf.xacro"/>
     <xacro:macro name="base_xacro" params="length radius">
         <link name="base_foot_print"/>
@@ -22,4 +23,5 @@
                 </material>
             </collision>
+            <xacro:cylinder_inertia m="1.0" r="${radius}" h="${length}"/>
         </link>
         <joint name="base_to_footprint_joint" type="fixed">

File: chapt6/chapt6_ws/src/fishbot_description/urdf/fishbot/actuator/caster.urdf.xacro (robot description, xacro)
@@ -1,4 +1,5 @@
 <?xml version="1.0"?>
 <robot xmlns:xacro="http://www.ros.org/wiki/xacro">
+    <xacro:include filename="$(find fishbot_description)/urdf/fishbot/common_inertia.urdf.xacro"/>
     <xacro:macro name="caster_xacro" params="caster_name xyz">
         <link name="${caster_name}_link">
@@ -21,4 +22,5 @@
                 </material>
             </collision>
+            <xacro:shpere_inertia m="0.05" r="0.016"/>
         </link>
         <joint name="${caster_name}_base_link_joint" type="fixed">

File: chapt6/chapt6_ws/src/fishbot_description/urdf/fishbot/actuator/wheel.urdf.xacro (robot description, xacro)
@@ -1,4 +1,5 @@
 <?xml version="1.0"?>
 <robot xmlns:xacro="http://www.ros.org/wiki/xacro">
+    <xacro:include filename="$(find fishbot_description)/urdf/fishbot/common_inertia.urdf.xacro"/>
     <xacro:macro name="wheel_xacro" params="wheel_name xyz">
         <link name="${wheel_name}_link">
@@ -21,4 +22,5 @@
                 </material>
             </collision>
+            <xacro:cylinder_inertia m="0.05" r="0.032" h="0.04"/>
         </link>
         <joint name="${wheel_name}_base_link_joint" type="continuous">

File: chapt6/chapt6_ws/src/fishbot_description/urdf/fishbot/sensor/camera.urdf.xacro (robot description, xacro)
@@ -1,4 +1,5 @@
 <?xml version="1.0"?>
 <robot xmlns:xacro="http://www.ros.org/wiki/xacro">
+    <xacro:include filename="$(find fishbot_description)/urdf/fishbot/common_inertia.urdf.xacro"/>
     <xacro:macro name="camera_xacro" params="xyz">
         <link name="camera_link">
@@ -21,4 +22,5 @@
                 </material>
             </collision>
+            <xacro:box_inertia m="0.1" w="0.02" h="0.10" d="0.02"/>
         </link>
         <!-- 关节用于组合部件 -->

File: chapt6/chapt6_ws/src/fishbot_description/urdf/fishbot/sensor/imu.urdf.xacro (robot description, xacro)
@@ -1,4 +1,5 @@
 <?xml version="1.0"?>
 <robot xmlns:xacro="http://www.ros.org/wiki/xacro">
+    <xacro:include filename="$(find fishbot_description)/urdf/fishbot/common_inertia.urdf.xacro"/>
     <xacro:macro name="imu_xacro" params="xyz">
         <link name="imu_link">
@@ -12,4 +13,16 @@
                 </material>
             </visual>
+        <collision>
+            <visual>
+                <origin xyz="0.0 0.0 0.0" rpy="0.0 0.0 0.0" />
+                <geometry>
+                    <box size="0.02 0.02 0.02" />
+                </geometry>
+                <material name="black">
+                    <color rgba="0.0 0.0 0.0 1.0" />
+                </material>
+            </visual>
+        </collision>
+        <xacro:box_inertia m="0.05" w="0.02" h="0.02" d="0.02"/>
         </link>
         <!-- 关节用于组合部件 -->

File: chapt6/chapt6_ws/src/fishbot_description/urdf/fishbot/sensor/laser.urdf.xacro (robot description, xacro)
@@ -1,4 +1,5 @@
 <?xml version="1.0"?>
 <robot xmlns:xacro="http://www.ros.org/wiki/xacro">
+    <xacro:include filename="$(find fishbot_description)/urdf/fishbot/common_inertia.urdf.xacro"/>
     <xacro:macro name="laser_xacro" params="xyz">
         <!-- 雷达支撑杆 -->

Commit message: 安装了差分驱动的插件

File: chapt6/chapt6_ws/install/fishbot_description/share/fishbot_description/urdf/fishbot/base.urdf.xacro (robot description, xacro)
@@ -26,5 +26,5 @@
         </link>
         <joint name="base_to_footprint_joint" type="fixed">
-            <origin xyz="0.0 0.0 ${length/2+0.032-0.001}" rpy="0.0 0.0 0.0" />
+            <origin xyz="0.0 0.0 ${length/2+0.032}" rpy="0.0 0.0 0.0" />
             <parent link="base_foot_print" />
             <child link="base_link" />

File: chapt6/chapt6_ws/install/fishbot_description/share/fishbot_description/urdf/fishbot/fishbot.urdf.xacro (robot description, xacro)
@@ -5,4 +5,5 @@
     <xacro:include filename="$(find fishbot_description)/urdf/fishbot/sensor/laser.urdf.xacro" />
     <xacro:include filename="$(find fishbot_description)/urdf/fishbot/sensor/imu.urdf.xacro" />
+    <xacro:include filename="$(find fishbot_description)/urdf/fishbot/plugins/gazebo_control_plugins.xacro" />
     <xacro:include filename="$(find fishbot_description)/urdf/fishbot/actuator/wheel.urdf.xacro" />
     <xacro:include filename="$(find fishbot_description)/urdf/fishbot/actuator/caster.urdf.xacro" />
@@ -15,3 +16,4 @@
     <xacro:caster_xacro caster_name="front_caster" xyz="0.08 0 -0.076" />
     <xacro:caster_xacro caster_name="back_caster" xyz="-0.08 0 -0.076" />
+    <xacro:gazebo_control_plugin/>
 </robot>
