Commit message: ros2_control编写和深度相机编写

File: chapt6/chapt6_ws/install/fishbot_description/share/fishbot_description/urdf/fishbot/fishbot.urdf.xacro (robot description, xacro)
@@ -9,4 +9,5 @@
     <xacro:include filename="$(find fishbot_description)/urdf/fishbot/actuator/wheel.urdf.xacro" />
     <xacro:include filename="$(find fishbot_description)/urdf/fishbot/actuator/caster.urdf.xacro" />
+    <xacro:include filename="$(find fishbot_description)/urdf/fishbot/fishbot_ros2_control.xacro" />
     <xacro:base_xacro length="0.12" radius="0.1" />
     <xacro:imu_xacro xyz="0 0 0.02" />
@@ -17,5 +18,6 @@
     <xacro:caster_xacro caster_name="front_caster" xyz="0.08 0 -0.076" />
     <xacro:caster_xacro caster_name="back_caster" xyz="-0.08 0 -0.076" />
-    <xacro:gazebo_control_plugin/>
+    <!-- <xacro:gazebo_control_plugin/> -->
+    <xacro:fishbot_ros2_control/>
     <xacro:gazebo_sensor_plugin/>
 </robot>

File: chapt6/chapt6_ws/install/fishbot_description/share/fishbot_description/urdf/fishbot/plugins/gazebo_sensor_plugins.xacro (robot description, xacro)
@@ -15,7 +15,6 @@
                 <visualize>true</visualize>
                 <update_rate>20</update_rate>
-                <!-- 相对laser_link的xyz rpy -->
                 <pose>0 0 0 0 0 0</pose>
-								<!-- 激光传感器配置 -->
+                <!-- 激光传感器配置 -->
                 <ray>
                     <!-- 设置扫描范围 -->
@@ -36,5 +35,4 @@
                     <!-- 设置噪声 -->
                     <noise>
-                        <!-- 正态分布 -->
                         <type>gaussian</type>
                         <mean>0.0</mean>
@@ -44,4 +42,100 @@
             </sensor>
         </gazebo>
+        <gazebo reference="imu_link">
+            <sensor name="imu_sensor" type="imu">
+                <plugin name="imu_plugin" filename="libgazebo_ros_imu_sensor.so">
+                    <ros>
+                        <namespace>/</namespace>
+                        <remapping>~/out:=imu</remapping>
+                    </ros>
+                    <!-- 这个不用初始化朝向作为参考系 -->
+                    <initial_orientation_as_reference>false</initial_orientation_as_reference>
+                </plugin>
+                <update_rate>100</update_rate>
+                <!-- 传感器始终打开 -->
+                <always_on>true</always_on>
+                <!-- 六轴噪声设置 -->
+                <imu>
+                    <angular_velocity>
+                        <x>
+                            <noise type="gaussian">
+                                <mean>0.0</mean>
+                                <stddev>2e-4</stddev>
+                                <bias_mean>0.0000075</bias_mean>
+                                <bias_stddev>0.0000008</bias_stddev>
+                            </noise>
+                        </x>
+                        <y>
+                            <noise type="gaussian">
+                                <mean>0.0</mean>
+                                <stddev>2e-4</stddev>
+                                <bias_mean>0.0000075</bias_mean>
+                                <bias_stddev>0.0000008</bias_stddev>
+                            </noise>
+                        </y>
+                        <z>
+                            <noise type="gaussian">
+                                <mean>0.0</mean>
+                                <stddev>2e-4</stddev>
+                                <bias_mean>0.0000075</bias_mean>
+                                <bias_stddev>0.0000008</bias_stddev>
+                            </noise>
+                        </z>
+                    </angular_velocity>
+                    <linear_acceleration>
+                        <x>
+                            <noise type="gaussian">
+                                <mean>0.0</mean>
+                                <stddev>1.7e-2</stddev>
+                                <bias_mean>0.1</bias_mean>
+                                <bias_stddev>0.001</bias_stddev>
+                            </noise>
+                        </x>
+                        <y>
+                            <noise type="gaussian">
+                                <mean>0.0</mean>
+                                <stddev>1.7e-2</stddev>
+                                <bias_mean>0.1</bias_mean>
+                                <bias_stddev>0.001</bias_stddev>
+                            </noise>
+                        </y>
+                        <z>
+                            <noise type="gaussian">
+                                <mean>0.0</mean>
+                                <stddev>1.7e-2</stddev>
+                                <bias_mean>0.1</bias_mean>
+                                <bias_stddev>0.001</bias_stddev>
+                            </noise>
+                        </z>
+                    </linear_acceleration>
+                </imu>
+            </sensor>
+        </gazebo>
     </xacro:macro>
+    <gazebo reference="camera_link">
+        <sensor type="depth" name="camera_sensor">
+            <plugin name="depth_camera" filename="libgazebo_ros_camera.so">
+                <!-- 固定到这个link上面 -->
+                <frame_name>camera_optical_link</frame_name>
+            </plugin>
+            <always_on>true</always_on>
+            <update_rate>100</update_rate>
+            <camera name="camera">
+                <horizontal_fov>1.5009831567</horizontal_fov>
+                <image>
+                    <width>800</width>
+                    <height>600</height>
+                    <format>R8G8B8</format>
+                </image>
+                <distortion>
+                    <k1>0.0</k1>
+                    <k2>0.0</k2>
+                    <k3>0.0</k3>
+                    <p1>0.0</p1>
+                    <p2>0.0</p2>
+                    <center>0.5 0.5</center>
+                </distortion>
+            </camera>
+        </sensor>
+    </gazebo>
 </robot>

File: chapt6/chapt6_ws/install/fishbot_description/share/fishbot_description/urdf/fishbot/sensor/camera.urdf.xacro (robot description, xacro)
@@ -3,4 +3,6 @@
     <xacro:include filename="$(find fishbot_description)/urdf/fishbot/common_inertia.urdf.xacro" />
     <xacro:macro name="camera_xacro" params="xyz">
+        <link name="camera_optical_link">
+        </link>
         <link name="camera_link">
             <visual>
@@ -33,4 +35,9 @@
             <material>Gazebo/Black</material>
         </gazebo>
+        <joint name="camera_optical_joint" type="fixed">
+            <parent link="camera_link"/>
+            <child link="camera_optical_link"/>
+            <origin xyz="0.0 0.0 0.0" rpy="${-pi/2} 0.0 ${-pi/2}"/>
+        </joint>
     </xacro:macro>
 </robot>
